File: Open Task Light/Electronics/Power Link/Source/Power Link.brd (EAGLE design)
At the start: 28.4 x 28.4 mm, 8 parts

Commit message: Control board PCB files + standardization
Parts:
- PIN1, PIN2, PIN3, PIN4, PIN5, PIN6, PIN7, PIN8: value OmniBall SMD Contact -> 0945-0-15-20-09-14-11-0
