File: Open Task Light/Electronics/Power Link/Source/Power Link.sch (EAGLE design)
At the start: 8 parts

Commit message: Control board PCB files + standardization
Parts:
- PIN1, PIN2, PIN3, PIN4, PIN5, PIN6, PIN7, PIN8: value OmniBall SMD Contact -> 0945-0-15-20-09-14-11-0
Changed lines of the file:
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@@
 </classes>
 <parts>
-<part name="PIN1" library="MILL_MAX_0945_SMD" library_urn="urn:adsk.wipprod:fs.file:vf.dSKtJUQlTnqB1DVnww3Itw" deviceset="0945-0-15-20-09-14-11-0" device="" value="OmniBall SMD Contact"/>
-<part name="PIN2" library="MILL_MAX_0945_SMD" library_urn="urn:adsk.wipprod:fs.file:vf.dSKtJUQlTnqB1DVnww3Itw" deviceset="0945-0-15-20-09-14-11-0" device="" value="OmniBall SMD Contact"/>
-<part name="PIN3" library="MILL_MAX_0945_SMD" library_urn="urn:adsk.wipprod:fs.file:vf.dSKtJUQlTnqB1DVnww3Itw" deviceset="0945-0-15-20-09-14-11-0" device="" value="OmniBall SMD Contact"/>
-<part name="PIN4" library="MILL_MAX_0945_SMD" library_urn="urn:adsk.wipprod:fs.file:vf.dSKtJUQlTnqB1DVnww3Itw" deviceset="0945-0-15-20-09-14-11-0" device="" value="OmniBall SMD Contact"/>
-<part name="PIN6" library="MILL_MAX_0945_SMD" library_urn="urn:adsk.wipprod:fs.file:vf.dSKtJUQlTnqB1DVnww3Itw" deviceset="0945-0-15-20-09-14-11-0" device="" value="OmniBall SMD Contact"/>
-<part name="PIN5" library="MILL_MAX_0945_SMD" library_urn="urn:adsk.wipprod:fs.file:vf.dSKtJUQlTnqB1DVnww3Itw" deviceset="0945-0-15-20-09-14-11-0" device="" value="OmniBall SMD Contact"/>
-<part name="PIN7" library="MILL_MAX_0945_SMD" library_urn="urn:adsk.wipprod:fs.file:vf.dSKtJUQlTnqB1DVnww3Itw" deviceset="0945-0-15-20-09-14-11-0" device="" value="OmniBall SMD Contact"/>
-<part name="PIN8" library="MILL_MAX_0945_SMD" library_urn="urn:adsk.wipprod:fs.file:vf.dSKtJUQlTnqB1DVnww3Itw" deviceset="0945-0-15-20-09-14-11-0" device="" value="OmniBall SMD Contact"/>
+<part name="PIN1" library="MILL_MAX_0945_SMD" library_urn="urn:adsk.wipprod:fs.file:vf.dSKtJUQlTnqB1DVnww3Itw" deviceset="0945-0-15-20-09-14-11-0" device="" value="0945-0-15-20-09-14-11-0"/>
+<part name="PIN2" library="MILL_MAX_0945_SMD" library_urn="urn:adsk.wipprod:fs.file:vf.dSKtJUQlTnqB1DVnww3Itw" deviceset="0945-0-15-20-09-14-11-0" device="" value="0945-0-15-20-09-14-11-0"/>
+<part name="PIN3" library="MILL_MAX_0945_SMD" library_urn="urn:adsk.wipprod:fs.file:vf.dSKtJUQlTnqB1DVnww3Itw" deviceset="0945-0-15-20-09-14-11-0" device="" value="0945-0-15-20-09-14-11-0"/>
+<part name="PIN4" library="MILL_MAX_0945_SMD" library_urn="urn:adsk.wipprod:fs.file:vf.dSKtJUQlTnqB1DVnww3Itw" deviceset="0945-0-15-20-09-14-11-0" device="" value="0945-0-15-20-09-14-11-0"/>
+<part name="PIN6" library="MILL_MAX_0945_SMD" library_urn="urn:adsk.wipprod:fs.file:vf.dSKtJUQlTnqB1DVnww3Itw" deviceset="0945-0-15-20-09-14-11-0" device="" value="0945-0-15-20-09-14-11-0"/>
+<part name="PIN5" library="MILL_MAX_0945_SMD" library_urn="urn:adsk.wipprod:fs.file:vf.dSKtJUQlTnqB1DVnww3Itw" deviceset="0945-0-15-20-09-14-11-0" device="" value="0945-0-15-20-09-14-11-0"/>
+<part name="PIN7" library="MILL_MAX_0945_SMD" library_urn="urn:adsk.wipprod:fs.file:vf.dSKtJUQlTnqB1DVnww3Itw" deviceset="0945-0-15-20-09-14-11-0" device="" value="0945-0-15-20-09-14-11-0"/>
+<part name="PIN8" library="MILL_MAX_0945_SMD" library_urn="urn:adsk.wipprod:fs.file:vf.dSKtJUQlTnqB1DVnww3Itw" deviceset="0945-0-15-20-09-14-11-0" device="" value="0945-0-15-20-09-14-11-0"/>
 </parts>
 <sheets>
