File: Open Task Light/Electronics/Power Track/Source/Power Track.brd (EAGLE design)
At the start: 10.8 x 432 mm, 3 parts, among them J1 220098-0271

Commit message: Control board PCB files + standardization
Parts:
- J1: value 220098-0271 -> 2200980271
- MP1: value WE-SMSA_3.3MMDEFAULT -> 78614025360; device ROUND SPACER M3 STEEL 2:WE-SMSA_78614020360 -> ROUND SPACER M3 STEEL 2.50MM:WE-SMSA_78614020360
Changed lines of the file:
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@@
 </attributes>
 <variantdefs>
+<variantdef name="Production"/>
 </variantdefs>
 <classes>
@@
 </autorouter>
 <elements>
-<element name="J1" library="molex-right-angle-220098-0271" library_urn="urn:adsk.wipprod:fs.file:vf.oH1rBRzZQjGkHvqZg5Po9g" package="2200980271" value="220098-0271" x="0" y="213.995" smashed="yes" rot="R180">
-<attribute name="ARROW_PART_NUMBER" value="" x="0" y="213.995" size="1.778" layer="27" rot="R180" display="off"/>
-<attribute name="ARROW_PRICE-STOCK" value="" x="0" y="213.995" size="1.778" layer="27" rot="R180" display="off"/>
-<attribute name="DESCRIPTION" value="Connector Header Through Hole, Right Angle 2 position 0.049&quot; (1.25mm)" x="0" y="213.995" size="1.778" layer="27" rot="R180" display="off"/>
-<attribute name="HEIGHT" value="4.05mm" x="0" y="213.995" size="1.778" layer="27" rot="R180" display="off"/>
+<element name="J1" library="molex-right-angle-220098-0271" library_urn="urn:adsk.wipprod:fs.file:vf.oH1rBRzZQjGkHvqZg5Po9g" package="2200980271" value="2200980271" base_value="2200980271" x="0" y="213.995" smashed="yes" rot="R180">
+<attribute name="DATASHEET" value="https://www.molex.com/en-us/products/part-detail-pdf/2200980271?display=pdf" x="0" y="213.995" size="1.778" layer="27" rot="R180" display="off"/>
 <attribute name="MANUFACTURER" value="Molex" x="0" y="213.995" size="1.778" layer="27" rot="R180" display="off"/>
-<attribute name="MOUSER_PART_NUMBER" value="538-220098-0271" x="0" y="213.995" size="1.778" layer="27" rot="R180" display="off"/>
-<attribute name="MOUSER_PRICE-STOCK" value="https://www.mouser.co.uk/ProductDetail/Molex/220098-0271?qs=mELouGlnn3fRzHRZ40buew%3D%3D" x="0" y="213.995" size="1.778" layer="27" rot="R180" display="off"/>
-<attribute name="MPN" value="220098-0271" x="0" y="213.995" size="1.778" layer="27" rot="R180" display="off"/>
+<attribute name="MPN" value="2200980271" x="0" y="213.995" size="1.778" layer="27" rot="R180" display="off"/>
 </element>
-<element name="MP1" library="ROUND SPACER M3 STEEL 2" library_urn="urn:adsk.wipprod:fs.file:vf.OljqTMRBRcqdr2rPhi7ygQ" package="WE-SMSA_78614020360" value="WE-SMSA_3.3MMDEFAULT" x="0" y="-211.06" smashed="yes" rot="MR180">
+<element name="MP1" library="ROUND SPACER M3 STEEL 2.50MM" library_urn="urn:adsk.wipprod:fs.file:vf.OljqTMRBRcqdr2rPhi7ygQ" package="WE-SMSA_78614020360" value="78614025360" base_value="78614025360" x="0" y="-211.06" smashed="yes" rot="MR180">
+<attribute name="DATASHEET" value="https://www.we-online.com/components/products/datasheet/78614025360.pdf" x="0" y="-211.06" size="1.778" layer="28" rot="MR180" display="off"/>
 <attribute name="DESCRIPTION" value="M3 solderable SMD standoff" x="0" y="-211.06" size="1.778" layer="28" rot="MR180" display="off"/>
 <attribute name="MANUFACTURER" value="Würth Elektronik" x="0" y="-211.06" size="1.778" layer="28" rot="MR180" display="off"/>
 <attribute name="MPN" value="78614025360" x="0" y="-211.06" size="1.778" layer="28" rot="MR180" display="off"/>
 </element>
-<element name="CONTACT_PADS" library="Power Track Pads" library_urn="urn:adsk.wipprod:fs.file:vf.ecLPPA_xR2C4rnfr6W4XRw" package="POWER-TRACK-PADS" value="POWERTRACKPAD" x="0" y="209.5" smashed="yes">
+<element name="CONTACT_PADS" library="Power Track Pads" library_urn="urn:adsk.wipprod:fs.file:vf.ecLPPA_xR2C4rnfr6W4XRw" package="POWER-TRACK-PADS" value="POWERTRACKPAD" base_value="POWERTRACKPAD" x="0" y="209.5" smashed="yes">
 </element>
 </elements>
