File: Open Task Light/Electronics/Power Track/Source/Power Track.sch (EAGLE design)
At the start: 3 parts, among them J1 220098-0271

Commit message: Control board PCB files + standardization
Parts:
- J1: value 220098-0271 -> 2200980271
- MP1: value WE-SMSA_3.3MMDEFAULT -> 78614025360; device ROUND SPACER M3 STEEL 2:WE-SMSA_3.3MMDEFAULT -> ROUND SPACER M3 STEEL 2.50MM:WE-SMSA_3.3MMDEFAULT
Changed lines of the file:
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@@
 </attributes>
 <variantdefs>
+<variantdef name="Production"/>
 </variantdefs>
 <classes>
@@
 </classes>
 <parts>
-<part name="J1" library="molex-right-angle-220098-0271" library_urn="urn:adsk.wipprod:fs.file:vf.oH1rBRzZQjGkHvqZg5Po9g" deviceset="220098-0271" device=""/>
-<part name="MP1" library="ROUND SPACER M3 STEEL 2" library_urn="urn:adsk.wipprod:fs.file:vf.OljqTMRBRcqdr2rPhi7ygQ" deviceset="WE-SMSA_3.3MM" device="DEFAULT"/>
-<part name="CONTACT_PADS" library="Power Track Pads" library_urn="urn:adsk.wipprod:fs.file:vf.ecLPPA_xR2C4rnfr6W4XRw" deviceset="POWERTRACKPAD" device="" value="POWERTRACKPAD"/>
+<part name="J1" library="molex-right-angle-220098-0271" library_urn="urn:adsk.wipprod:fs.file:vf.oH1rBRzZQjGkHvqZg5Po9g" deviceset="220098-0271" device="" value="2200980271"/>
+<part name="MP1" library="ROUND SPACER M3 STEEL 2.50MM" library_urn="urn:adsk.wipprod:fs.file:vf.OljqTMRBRcqdr2rPhi7ygQ" deviceset="WE-SMSA_3.3MM" device="DEFAULT" value="78614025360"/>
+<part name="CONTACT_PADS" library="Power Track Pads" library_urn="urn:adsk.wipprod:fs.file:vf.ecLPPA_xR2C4rnfr6W4XRw" deviceset="POWERTRACKPAD" device="" value="POWERTRACKPAD">
+<variant name="Production" populate="no"/>
+</part>
 </parts>
 <sheets>
@@
 <instances>
 <instance part="J1" gate="G$1" x="-35.56" y="0" smashed="yes" rot="R180">
-<attribute name="NAME" x="-52.07" y="-7.62" size="1.778" layer="95" rot="R180" align="center-left"/>
-<attribute name="VALUE" x="-52.07" y="-5.08" size="1.778" layer="96" rot="R180" align="center-left"/>
+<attribute name="NAME" x="-36.83" y="-2.54" size="1.778" layer="95" rot="R180" align="center-left"/>
+<attribute name="VALUE" x="-52.07" y="-5.08" size="1.778" layer="96" rot="R180" align="center-left" display="off"/>
 </instance>
 <instance part="MP1" gate="G$1" x="5.08" y="-22.86" smashed="yes">
@@
 <wire x1="-35.56" y1="0" x2="-15.24" y2="0" width="0.1524" layer="91"/>
 <wire x1="-15.24" y1="0" x2="-15.24" y2="-2.54" width="0.1524" layer="91"/>
+<pinref part="J1" gate="G$1" pin="1"/>
 <pinref part="CONTACT_PADS" gate="G$1" pin="24V"/>
-<pinref part="J1" gate="G$1" pin="1"/>
 </segment>
 </net>
@@
 <wire x1="-35.56" y1="2.54" x2="-15.24" y2="2.54" width="0.1524" layer="91"/>
 <wire x1="-15.24" y1="2.54" x2="-15.24" y2="5.08" width="0.1524" layer="91"/>
+<pinref part="J1" gate="G$1" pin="2"/>
 <pinref part="CONTACT_PADS" gate="G$1" pin="GND"/>
-<pinref part="J1" gate="G$1" pin="2"/>
 </segment>
 </net>
