File: Open Task Light/Electronics/Control Board/Source/Control Board.brd (EAGLE design)
At the start: 48 x 115 mm, 25 parts, among them U1 TS12A4515D

Commit message: Control board gerber bottom layer fix (#60)
Added bottom copper layer to Gerbers which was excluded from Fusion export
Clean up top silkscreen to remove big `HEADER` labels
Parts:
- RECOM-BUCK: device R-78K5.0-1.0:R-78K5.0-1.0_RCP -> R-78K5.0-1:R-78K5.0-1.0_RCP
- RECOM-DRIVER: device [DRIVER]RCD-24-0.70_Vref:RCD24030 -> [DRIVER]RCD-24-0:RCD24030
- U$2: device 2.5mm-plated-through-hole:2.5MMPLATEDHOLE -> 2:2.5MMPLATEDHOLE
Changed lines of the file:
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@@
 <grid distance="0.25" unitdist="mm" unit="mm" style="lines" multiple="1" display="yes" altdistance="5" altunitdist="mil" altunit="mil"/>
 <layers>
-<layer number="1" name="Top" color="4" fill="1" visible="yes" active="yes"/>
+<layer number="1" name="Top" color="4" fill="1" visible="no" active="yes"/>
 <layer number="2" name="Route2" color="16" fill="1" visible="no" active="no"/>
 <layer number="3" name="Route3" color="17" fill="1" visible="no" active="no"/>
@@
 <layer number="14" name="Route14" color="22" fill="1" visible="no" active="no"/>
 <layer number="15" name="Route15" color="23" fill="1" visible="no" active="no"/>
-<layer number="16" name="Bottom" color="1" fill="1" visible="yes" active="yes"/>
-<layer number="17" name="Pads" color="2" fill="1" visible="yes" active="yes"/>
-<layer number="18" name="Vias" color="2" fill="1" visible="yes" active="yes"/>
-<layer number="19" name="Unrouted" color="6" fill="1" visible="yes" active="yes"/>
-<layer number="20" name="Dimension" color="24" fill="1" visible="yes" active="yes"/>
+<layer number="16" name="Bottom" color="1" fill="1" visible="no" active="yes"/>
+<layer number="17" name="Pads" color="2" fill="1" visible="no" active="yes"/>
+<layer number="18" name="Vias" color="2" fill="1" visible="no" active="yes"/>
+<layer number="19" name="Unrouted" color="6" fill="1" visible="no" active="yes"/>
+<layer number="20" name="Dimension" color="24" fill="1" visible="no" active="yes"/>
 <layer number="21" name="tPlace" color="7" fill="1" visible="yes" active="yes"/>
 <layer number="22" name="bPlace" color="7" fill="1" visible="yes" active="yes"/>
@@
 <layer number="43" name="vRestrict" color="2" fill="10" visible="no" active="yes"/>
 <layer number="44" name="Drills" color="7" fill="1" visible="no" active="yes"/>
-<layer number="45" name="Holes" color="7" fill="1" visible="yes" active="yes"/>
+<layer number="45" name="Holes" color="7" fill="1" visible="no" active="yes"/>
 <layer number="46" name="Milling" color="3" fill="1" visible="no" active="yes"/>
 <layer number="47" name="Measures" color="7" fill="1" visible="no" active="yes"/>
@@
 <layer number="196" name="mValues" color="7" fill="1" visible="no" active="yes"/>
 <layer number="199" name="Contour" color="7" fill="1" visible="no" active="yes"/>
-<layer number="200" name="PrivateNotes" color="7" fill="1" visible="yes" active="yes"/>
+<layer number="200" name="PrivateNotes" color="7" fill="1" visible="no" active="yes"/>
 <layer number="201" name="201bmp" color="7" fill="1" visible="no" active="no"/>
 <layer number="202" name="202bmp" color="7" fill="1" visible="no" active="no"/>
@@
 <attribute name="MPN" value="807-22-001-10-001101" x="0" y="-35" size="1.778" layer="28" rot="MR0" display="off"/>
 </element>
-<element name="RECOM-DRIVER" library="[DRIVER]RCD-24-0.70_Vref" library_urn="urn:adsk.wipprod:fs.file:vf.xL-8JYjTRVy-J5S12aLTOQ" package="RCD24030" value="RCD-24-0.70/VREF" base_value="RCD-24-0.70/VREF" x="8.2926" y="-12.8125" smashed="yes" rot="R90">
+<element name="RECOM-DRIVER" library="[DRIVER]RCD-24-0" library_urn="urn:adsk.wipprod:fs.file:vf.xL-8JYjTRVy-J5S12aLTOQ" package="RCD24030" value="RCD-24-0.70/VREF" base_value="RCD-24-0.70/VREF" x="8.2926" y="-12.8125" smashed="yes" rot="R90">
 <attribute name="DATASHEET" value="https://recom-power.com/pdf/Lightline_DC-DC/RCD-24.pdf" x="8.2926" y="-12.8125" size="1.778" layer="27" rot="R90" display="off"/>
 <attribute name="MANUFACTURER" value="RECOM Power" x="8.2926" y="-12.8125" size="1.778" layer="27" rot="R90" display="off"/>
@@
 <attribute name="NAME" x="11.7276" y="-2.7975" size="1.016" layer="25" font="custom" fontFamily="Chivo Mono" rot="R90" align="center"/>
 </element>
-<element name="RECOM-BUCK" library="R-78K5.0-1.0" library_urn="urn:adsk.wipprod:fs.file:vf.2k1aaWgXQseguvClFT_OyA" package="R-78K5.0-1.0_RCP" value="R-78K5.0-1.0" base_value="R-78K5.0-1.0" x="11.3956" y="10.8642" smashed="yes" rot="R90">
+<element name="RECOM-BUCK" library="R-78K5.0-1" library_urn="urn:adsk.wipprod:fs.file:vf.2k1aaWgXQseguvClFT_OyA" package="R-78K5.0-1.0_RCP" value="R-78K5.0-1.0" base_value="R-78K5.0-1.0" x="11.3956" y="10.8642" smashed="yes" rot="R90">
 <attribute name="DATASHEET" value="https://recom-power.com/pdf/Innoline/R-78K-1.0.pdf" x="11.3956" y="10.8642" size="1.778" layer="27" rot="R90" display="off"/>
 <attribute name="MANUFACTURER" value="RECOM Power" x="11.3956" y="10.8642" size="1.778" layer="27" rot="R90" display="off"/>
@@
 <attribute name="MPN" value="2200980271" x="0" y="-72.625" size="1.778" layer="27" display="off"/>
 </element>
-<element name="U$2" library="2.5mm-plated-through-hole" library_urn="urn:adsk.wipprod:fs.file:vf.mf-xDpjkSn6krzUzkZIXjA" package="2.5MMPLATEDHOLE" value="2.5MMPLATEDTHROUGHHOLE" x="0" y="-88.742" locked="yes" smashed="yes">
+<element name="U$2" library="2" library_urn="urn:adsk.wipprod:fs.file:vf.mf-xDpjkSn6krzUzkZIXjA" package="2.5MMPLATEDHOLE" value="2.5MMPLATEDTHROUGHHOLE" x="0" y="-88.742" locked="yes" smashed="yes">
 </element>
 <element name="RES5.6K1" library="RC1206JR-075K6L" library_urn="urn:adsk.wipprod:fs.file:vf.xNELdiplRwS8PI3aTA94vQ" package="RESC3116X65N" value="RC1206JR-075K6L" base_value="RC1206JR-075K6L" x="-12" y="-14" smashed="yes" rot="R180">
@@
 <attribute name="MANUFACTURER" value="Nexperia" x="1.5" y="-14.5" size="1.778" layer="27" rot="R90" display="off"/>
 <attribute name="MPN" value="PMEG4010EGWX" x="1.5" y="-14.5" size="1.778" layer="27" rot="R90" display="off"/>
-<attribute name="NAME" x="-0.024" y="-17.04" size="1.32" layer="25" ratio="10" rot="R90"/>
+<attribute name="NAME" x="1.226" y="-15.04" size="0.55" layer="25" ratio="10" rot="R90"/>
 </element>
 <element name="D1" library="Diodes" library_urn="urn:adsk.wipprod:fs.file:vf.ReqFR3WWTOaeHyFqncs7zQ" package="SOD-123" package3d_urn="urn:adsk.eagle:package:10898395/2" value="PMEG4010EGWX" base_value="PMEG4010EGWX" x="-18.75" y="8" smashed="yes" rot="R90">
@@
 <attribute name="MANUFACTURER" value="Nexperia" x="-18.75" y="8" size="1.778" layer="27" rot="R90" display="off"/>
 <attribute name="MPN" value="PMEG4010EGWX" x="-18.75" y="8" size="1.778" layer="27" rot="R90" display="off"/>
-<attribute name="NAME" x="-20.274" y="5.46" size="1.32" layer="25" ratio="10" rot="R90"/>
+<attribute name="NAME" x="-19.024" y="7.46" size="0.55" layer="25" ratio="10" rot="R90"/>
 </element>
 <element name="FUSE" library="SMD2016B100TF/33" library_urn="urn:adsk.wipprod:fs.file:vf.DudsQ56ZSC6e9TcR25F48g" package="SMD2016B100TF/33" value="SMD2016B100TF/33" base_value="SMD2016B100TF/33" x="0" y="-65.375" smashed="yes" rot="R90">
@@
 <attribute name="MANUFACTURER" value="Samtec" x="-11.4524" y="3.7642" size="1.778" layer="27" rot="R270" display="off"/>
 <attribute name="MPN" value="CES-107-01-G-S" x="-11.4524" y="3.7642" size="1.778" layer="27" rot="R270" display="off"/>
-<attribute name="NAME" x="-8.743390625" y="19.9352" size="1.905" layer="25" rot="R270"/>
-<attribute name="VALUE" x="-12.1524" y="3.7642" size="0.635" layer="27" rot="R270" align="bottom-center"/>
 </element>
 <element name="HEADER2" library="SAMTEC-CES-107-01-X-S" library_urn="urn:adsk.wipprod:fs.file:vf.xCfvTjADSDSlnBbDXrn8DA" package="SAMTEC-CES-107-01-X-S" value="CES-107-01-G-S" base_value="CES-107-01-G-S" x="3.7876" y="3.7642" smashed="yes" rot="R90">
@@
 <attribute name="MANUFACTURER" value="Samtec" x="3.7876" y="3.7642" size="1.778" layer="27" rot="R90" display="off"/>
 <attribute name="MPN" value="CES-107-01-G-S" x="3.7876" y="3.7642" size="1.778" layer="27" rot="R90" display="off"/>
-<attribute name="NAME" x="1.078590625" y="-12.4068" size="1.905" layer="25" rot="R90"/>
-<attribute name="VALUE" x="4.4876" y="3.7642" size="0.635" layer="27" rot="R90" align="bottom-center"/>
 </element>
 </elements>
